Commit message: curriculum

File: gym_pybullet_drones/assets/gate.urdf (robot description, URDF)
Before this commit: robot gate, 1 links, 0 joints
Links:
- link base_link: geometry visual mesh filename=./assets/gate.obj scale=.04 .04 .04

Commit message: fix

File: gym_pybullet_drones/assets/gate.urdf (robot description, URDF)
Before this commit: robot gate, 1 links, 0 joints
Links:
- link base_link: geometry visual mesh filename=./assets/gate.obj scale=.02 .02 .02

Commit message: add_curriculum_and_ddpg

File: gym_pybullet_drones/assets/gate.urdf (robot description, URDF)
Before this commit: robot gate, 1 links, 0 joints
Links:
- link base_link: geometry visual mesh filename=./assets/gate.obj scale=.018 .018 .018

Commit message: fix_env_and_reward_function

File: gym_pybullet_drones/assets/gate.urdf (robot description, URDF)
Before this commit: robot gate, 1 links, 0 joints
Links:
- link base_link: geometry collision box size=0.012 0.038042 0.085716; collision box size=0.012 0.038042 0.085716
